File: Charger.sch (KiCad schematic (older format))
At the start: 1 part

Commit message: Worked on Charger
Parts:
- added C? (x2): 0u01, symbol C_Small
- added C? (x3): 0u1, symbol C_Small
- added C? (x2): 1u, symbol C_Small
- added D? (x2): D_Schottky, symbol D_Schottky_Small
- added R?: 1k, symbol R_Small
- added R? (x2): 59k 1%, symbol R_Small
- added R?: 19.6k 1%, symbol R_Small
- gave numbers to parts that had none: 1
Connections:
- net labels added: Charge-DCIN, Charge-Out, GNDPWR, ICTL, ~ACOK, ~SHDN
- wire segments 0 -> 38
Other:
- note added: "CELLS connected to VREFIN\nto set 4 cell charging"
- note added: "~SHDN\nis a digital input that stops\ncharging output. Connect to a digital\noutput\nICTL\nis an analog input to\ncontrol charging current.\n"
- moved on the sheet: U6
