File: Controller.sch (KiCad schematic (older format))
At the start: 61 parts

Commit message: mostly finished controller. Still need to decide on integration
Parts:
- removed C? (x2): 47n, symbol C_Small
- removed D?: V10P10, symbol SCHDPAK
- removed Q? (x3): NMOS_GSD_Body-Diode, symbol NMOS_GSD_Body-Diode
- removed Q?: Q_PMOS_GSD_Body_Diode, symbol Q_PMOS_GSD_Body_Diode
- removed R? (x2): 1k, symbol R_Small
- removed R? (x4): 10k, symbol R_Small
- removed R? (x4): 100/1W, symbol R_Small
- removed R? (x4): 330k, symbol R_Small
- added C?: 2u2, symbol C_Small
- added C?: 1u, symbol C_Small
- added D?: MMBD7000, TO_SOT_Packages_SMD:SOT-23, symbol MMBD7000
- added D?: V10P10, TO_SOT_Packages_SMD:TO-277A, symbol V10P10
- added D? (x4): SMAJ40CA, symbol TVS
- added D? (x3): 18V, symbol ZENERsmall
- added D? (x3): 43V, symbol ZENERsmall
- added D? (x2): PMEG6002, symbol ZENERsmall
- added D?: 3v3, symbol ZENERsmall
- added P?: XTR-Batt-10k, symbol CONN_01X02
- added Q? (x2): IRF1010E, TO_SOT_Packages_THT:TO-220_Horizontal, symbol IRF1010E
- added Q?: FDD8451, TO_SOT_Packages_SMD:TO-252-2Lead, symbol FDD8451
- added R? (x3): 10k, symbol R_Small
- added R? (x2): 22k, symbol R_Small
- added R? (x2): 0.002Ω @ 1W, symbol R_Small
- added R? (x5): 1M, symbol R_Small
- added R? (x2): 0, symbol R_Small
- added R? (x3): 3.3M, symbol R_Small
- added R?: 549k, symbol R_Small
- added R?: 200 @ 1W, symbol R_Small
- added R? (x5): 100, symbol R_Small
- added R? (x2): 499, symbol R_Small
- added R?: 1k, symbol R_Small
- added R?: 120k, symbol R_Small
- added R? (x2): 4k7, symbol R_Small
- added RT?: XTR-DCRG-FET-10k, symbol Thermistor-Small
- added SW?: Wakeup, symbol SW_PUSH_SMALL_H
- added SW?: FETSOFF, symbol SW_PUSH_SMALL_H
- added U?: USBLC6-2, TO_SOT_Packages_SMD:SOT-666, symbol USBLC6-2
- added U? (x2): SI1970, TO_SOT_Packages_SMD:SOT-363_SC-70-6_Handsoldering, symbol SI1970
Connections:
- net CFET: now also R?.1
- net DFET: now also R?.1
- net GNDPWR: now also C?.2, C?.2, U?.24 (ADDR), C?.1, C?.2, D?.2 (A), D?.2 (A), D?.2 (A), D?.2 (A), P?.2 (P2), R?.1, R?.1, R?.1, R?.1, R?.1, RT?.2, U?.2 (GND); no longer C?.1, C?.1
- net PCFET: now also R?.1
- net VDD: now also D?.1 (K), D?.1 (K)
- net at U?.10 (CB4): now also C?.2, R?.1, U?.11 (VC3), U?.6 (CB6), U?.7 (VC5), U?.8 (CB5), U?.9 (VC4)
- net at U?.12 (CB3): now also C?.2, R?.1, U?.13 (VC2)
- net Charger/Load-: now reaches C?.2, R?.1, U?.17 (VC0)
- net at U?.20 (XT1): now also P?.1 (P1), R?.1, R?.2
- net at U?.21 (XT2): now also R?.1, R?.2, RT?.1
- net at U?.22 (TEMPO): now also R?.2, R?.2
- net at U?.25 (SCL): now also R?.2, U?.4 (S2)
- net at U?.26 (SDAI): now also U?.27 (SDAO), R?.2, U?.1 (S2)
- net ~INT: now reaches U?.31 (~INT)
- net PSD: now reaches U?.32 (PSD)
- net FETSOFF: now reaches U?.33 (FETSOFF)
- net FETSOFF: now also C?.2, R?.2, R?.2
- net ~SD: now reaches U?.34 (~SD)
- net ~SD: now also R?.2
- net ~EOC: now reaches U?.35 (~EOC)
- net ~EOC: now also R?.2
- net RGO: now reaches U?.36 (RGO)
- net RGO: now also C?.1, D?.1 (K), R?.1, R?.1, R?.1, R?.1, SW?.1, U?.2 (G2), U?.5 (G2), U?.5 (VBUS)
- net CHMON: now reaches U?.37 (CHMON)
- net CHMON: now also R?.2
- net LDMON: now reaches U?.38 (LDMON)
- net LDMON: now also R?.1, R?.2
- net at C?.2: now also C?.1, R?.2; no longer U?.46 (CSI2)
- net +BATT: now reaches C?.2, R?.1, U?.48 (VBATT)
- net +BATT: now also D?.1, D?.1 (K), D?.2, D?.2 (A), R?.1, R?.2, R?.2, SW?.2
- new net: C?.1, C?.1, R?.2
- new net: D?.2 (A), D?.2 (A), D?.3, Q?.3 (S), Q?.3 (S), R?.1, R?.1, R?.1, R?.2, R?.2, R?.2
- new net: D?.1 (K), Q?.1 (G), R?.1, R?.2 (x3)
- new net: D?.1 (K), D?.2 (A), D?.3 (K), Q?.2 (D), Q?.2 (D), R?.2
- new net: D?.2 (A), Q?.3 (S), R?.1, R?.2
- new net: R?.2, U?.1 (I/O1)
- new net: R?.2, U?.3 (I/O2)
- new net: U?.3 (D2), U?.4 (I/O1)
- new net: U?.6 (D2), U?.6 (I/O2)
- new net: R?.2, SW?.1
- new net: R?.1, SW?.2
- new net CSI1: U?.47 (CSI1)
- new net CSI2: U?.46 (CSI2)
- new net Charger+: D?.1 (A), D?.2 (A), R?.1, R?.1, R?.1, R?.2, R?.2
- new net Load+: D?.1 (K), Q?.2 (D), R?.1, R?.2
- new net SCL: R?.1
- new net SDA: R?.1
Other:
- note added: "ADR tied to ground\nfor address 0. No\nneed to change it\nin normal opperation"
- note added: "May not populate.\nIf microcontroller used,\nthen this pin is driven\nby microcontroller or\nother protection circuit."
- note added: "Provide connections for\nboth off-board connection\nand microcontroller\ncontrol of SCL and SDA"
- note added: "XTR-Batt is an external connection\nfor thermistor to monitor battery temperature.\n\nXTR-DCRG-FET is an on-board thermistor \nmounted next to the discharge FET."
- moved on the sheet: C?, Q?, R?, U?

Commit message: These uncommitted files have been bugging me for waay tooo long
Parts:
- removed D? (x3): SMAJ40CA, symbol TVS
- added D3, D8: TVS, symbol TVS
- D?: symbol TVS -> TVS-RESCUE-portable-liIon-battery-pack
- gave numbers to parts that had none: 92
Connections:
- net +BATT: now also D3.1
- net GNDPWR: now also D?.1, D3.2, D8.1
- net Load+: now also D8.2
- net RGO: now also U4.2 (G2), U4.5 (G2); no longer U4.2 (G2), U4.5 (G2)
- net at R45.2, U3.25 (SCL): now also U4.1 (S2); no longer U4.4 (S2)
- net at R46.2, U3.26 (SDAI), U3.27 (SDAO): now also U4.4 (S2); no longer U4.1 (S2)
- net at D11.3 (K), D12.2 (A), D9.1 (K)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: now also D?.2
- net at U5.4 (I/O1): now also U4.6 (D2); no longer U4.3 (D2)
- net at U5.6 (I/O2): now also U4.3 (D2); no longer U4.6 (D2)
- net Charger/Load-: no longer names the net of C4.2, R32.1, U3.17 (VC0)
