File: Protection.sch (KiCad schematic (older format))
At the start: 1 part

Commit message: These uncommitted files have been bugging me for waay tooo long
Parts:
- added C? (x6): 0u1, symbol C_Small
- added R? (x4): 1k, symbol R_Small
- added R?: 100, symbol R_Small
- gave numbers to parts that had none: 1
Connections:
- net labels added: GNDPWR, OUT
- wire segments 10 -> 31
